File: HARDWARE/sensor/Hooly 2.023 0603/Hooly_2.023.sch (EAGLE design)
At the start: 34 parts, among them IC2 MCP1703CB, U3 MCP73831, U5 ATMEGA328P-AU

Commit message: Hardware update
Parts:
- removed U$6: FTDI232, My_library:FTDI232
- added SJ1, SJ2: (no value), jumper:SJ
- added U$5: FTDI232, My_library:FTDI232
- C12: value (none) -> 1uF
Connections:
- net DTR: now also U$5.DTR, U$7.D-; no longer U$6.DTR
- net GND: now also SJ1.2, SJ2.2, U$5.GND; no longer U$6.GND
- net RX: now also U$5.TX, U$7.D+; no longer U$6.TX
- net SW1: now also SJ1.1
- net SW2: now also SJ2.1
- net TX: now also U$5.RX, U$7.ID; no longer U$6.RX
- net VCC: now also U$5.VCC; no longer U$6.VCC
Changed lines of the file:
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@@
 <classes>
 <class number="0" name="default" width="0" drill="0">
+<clearance class="0" value="0.381"/>
 </class>
 </classes>
@@
 <part name="C8" library="resistor" library_urn="urn:adsk.eagle:library:348" deviceset="C-EU" device="C0603" package3d_urn="urn:adsk.eagle:package:26138/1" value=".1uF"/>
 <part name="SUPPLY16" library="supply2" library_urn="urn:adsk.eagle:library:372" deviceset="GND" device=""/>
-<part name="U$6" library="My_library" deviceset="FTDI232" device=""/>
 <part name="U$3" library="My_library" deviceset="MYDS18B20" device=""/>
 <part name="SUPPLY12" library="supply2" library_urn="urn:adsk.eagle:library:372" deviceset="VCC" device=""/>
@@
 <part name="C9" library="resistor" library_urn="urn:adsk.eagle:library:348" deviceset="C-US" device="C1206K" package3d_urn="urn:adsk.eagle:package:26202/1" value="1uF"/>
 <part name="C10" library="resistor" library_urn="urn:adsk.eagle:library:348" deviceset="C-US" device="C1206K" package3d_urn="urn:adsk.eagle:package:26202/1" value="1uF"/>
-<part name="C12" library="resistor" library_urn="urn:adsk.eagle:library:348" deviceset="C-US" device="C1206K" package3d_urn="urn:adsk.eagle:package:26202/1"/>
+<part name="C12" library="resistor" library_urn="urn:adsk.eagle:library:348" deviceset="C-US" device="C1206K" package3d_urn="urn:adsk.eagle:package:26202/1" value="1uF"/>
 <part name="Q1" library="crystal-geyer_V1_0" library_urn="urn:adsk.eagle:library:203" deviceset="KX" device="-9B" package3d_urn="urn:adsk.eagle:package:11930/1"/>
 <part name="C1" library="rcl" library_urn="urn:adsk.eagle:library:334" deviceset="C-EU" device="C0603K" package3d_urn="urn:adsk.eagle:package:23680/2"/>
 <part name="C3" library="rcl" library_urn="urn:adsk.eagle:library:334" deviceset="C-EU" device="C0603K" package3d_urn="urn:adsk.eagle:package:23680/2"/>
+<part name="U$5" library="My_library" deviceset="FTDI232" device=""/>
+<part name="SJ1" library="jumper" library_urn="urn:adsk.eagle:library:252" deviceset="SJ" device="" package3d_urn="urn:adsk.eagle:package:15471/1"/>
+<part name="SJ2" library="jumper" library_urn="urn:adsk.eagle:library:252" deviceset="SJ" device="" package3d_urn="urn:adsk.eagle:package:15471/1"/>
+<part name="GND1" library="supply2" library_urn="urn:adsk.eagle:library:372" deviceset="GND" device=""/>
 </parts>
 <sheets>
@@
 <instance part="C8" gate="G$1" x="127" y="60.96"/>
 <instance part="SUPPLY16" gate="GND" x="124.46" y="101.6"/>
-<instance part="U$6" gate="G$1" x="147.32" y="43.18"/>
 <instance part="U$3" gate="G$1" x="101.6" y="81.28" smashed="yes"/>
 <instance part="SUPPLY12" gate="G$1" x="50.8" y="127"/>
@@
 <attribute name="VALUE" x="134.239" y="113.284" size="1.778" layer="96" rot="R90"/>
 </instance>
+<instance part="U$5" gate="G$1" x="149.86" y="43.18"/>
+<instance part="SJ1" gate="1" x="139.7" y="91.44"/>
+<instance part="SJ2" gate="1" x="139.7" y="83.82"/>
+<instance part="GND1" gate="GND" x="147.32" y="76.2"/>
 </instances>
 <busses>
@@
 </segment>
 <segment>
-<pinref part="U$6" gate="G$1" pin="GND"/>
-<wire x1="137.16" y1="40.64" x2="119.38" y2="40.64" width="0.1524" layer="91"/>
+<wire x1="139.7" y1="40.64" x2="119.38" y2="40.64" width="0.1524" layer="91"/>
 <pinref part="SUPPLY14" gate="GND" pin="GND"/>
 <wire x1="119.38" y1="40.64" x2="119.38" y2="38.1" width="0.1524" layer="91"/>
+<pinref part="U$5" gate="G$1" pin="GND"/>
 </segment>
 <segment>
@@
 <pinref part="SUPPLY13" gate="GND" pin="GND"/>
 <wire x1="50.8" y1="101.6" x2="50.8" y2="96.52" width="0.1524" layer="91"/>
+</segment>
+<segment>
+<pinref part="SJ2" gate="1" pin="2"/>
+<wire x1="144.78" y1="83.82" x2="147.32" y2="83.82" width="0.1524" layer="91"/>
+<pinref part="GND1" gate="GND" pin="GND"/>
+<wire x1="147.32" y1="83.82" x2="147.32" y2="78.74" width="0.1524" layer="91"/>
+<pinref part="SJ1" gate="1" pin="2"/>
+<wire x1="144.78" y1="91.44" x2="147.32" y2="91.44" width="0.1524" layer="91"/>
+<wire x1="147.32" y1="91.44" x2="147.32" y2="83.82" width="0.1524" layer="91"/>
+<junction x="147.32" y="83.82"/>
 </segment>
 </net>
@@
 <pinref part="SUPPLY15" gate="G$1" pin="VCC"/>
 <wire x1="119.38" y1="55.88" x2="119.38" y2="43.18" width="0.1524" layer="91"/>
-<pinref part="U$6" gate="G$1" pin="VCC"/>
-<wire x1="119.38" y1="43.18" x2="137.16" y2="43.18" width="0.1524" layer="91"/>
+<wire x1="119.38" y1="43.18" x2="139.7" y2="43.18" width="0.1524" layer="91"/>
+<pinref part="U$5" gate="G$1" pin="VCC"/>
 </segment>
 <segment>
@@
 </segment>
 <segment>
-<pinref part="U$6" gate="G$1" pin="RX"/>
-<wire x1="137.16" y1="50.8" x2="129.54" y2="50.8" width="0.1524" layer="91"/>
+<wire x1="139.7" y1="50.8" x2="129.54" y2="50.8" width="0.1524" layer="91"/>
 <label x="129.54" y="50.8" size="1.778" layer="95"/>
+<pinref part="U$5" gate="G$1" pin="RX"/>
+</segment>
+<segment>
+<pinref part="U$7" gate="G$1" pin="ID"/>
+<wire x1="-30.48" y1="27.94" x2="-38.1" y2="27.94" width="0.1524" layer="91"/>
+<label x="-38.1" y="27.94" size="1.778" layer="95"/>
 </segment>
 </net>
@@
 <pinref part="C8" gate="G$1" pin="2"/>
 <wire x1="127" y1="55.88" x2="127" y2="45.72" width="0.1524" layer="91"/>
-<pinref part="U$6" gate="G$1" pin="DTR"/>
-<wire x1="127" y1="45.72" x2="137.16" y2="45.72" width="0.1524" layer="91"/>
+<wire x1="127" y1="45.72" x2="139.7" y2="45.72" width="0.1524" layer="91"/>
+<pinref part="U$5" gate="G$1" pin="DTR"/>
+</segment>
+<segment>
+<pinref part="U$7" gate="G$1" pin="D-"/>
+<wire x1="-30.48" y1="33.02" x2="-38.1" y2="33.02" width="0.1524" layer="91"/>
+<label x="-38.1" y="33.02" size="1.778" layer="95"/>
 </segment>
 </net>
@@
 </segment>
 <segment>
-<pinref part="U$6" gate="G$1" pin="TX"/>
-<wire x1="137.16" y1="48.26" x2="129.54" y2="48.26" width="0.1524" layer="91"/>
+<wire x1="139.7" y1="48.26" x2="129.54" y2="48.26" width="0.1524" layer="91"/>
 <label x="129.54" y="48.26" size="1.778" layer="95"/>
+<pinref part="U$5" gate="G$1" pin="TX"/>
+</segment>
+<segment>
+<pinref part="U$7" gate="G$1" pin="D+"/>
+<wire x1="-30.48" y1="30.48" x2="-38.1" y2="30.48" width="0.1524" layer="91"/>
+<label x="-38.1" y="30.48" size="1.778" layer="95"/>
 </segment>
 </net>
@@
 <label x="17.78" y="45.72" size="1.778" layer="95"/>
 </segment>
+<segment>
+<pinref part="SJ1" gate="1" pin="1"/>
+<wire x1="134.62" y1="91.44" x2="129.54" y2="91.44" width="0.1524" layer="91"/>
+<label x="127" y="91.44" size="1.778" layer="95"/>
+</segment>
 </net>
 <net name="SW2" class="0">
@@
 <label x="17.78" y="43.18" size="1.778" layer="95"/>
 </segment>
-</net>
+<segment>
+<pinref part="SJ2" gate="1" pin="1"/>
+<wire x1="134.62" y1="83.82" x2="129.54" y2="83.82" width="0.1524" layer="91"/>
+<label x="127" y="83.82" size="1.778" layer="95"/>
+</segment>
+</net>
